File: MAIN_CONTROLLER/MAIN_CONTROLLER.kicad_sch (KiCad schematic)
At the start: 0 parts

Commit message: Schematic Update
Parts:
- added C1, C2: 22pF, symbol Device:C
- added C10: 106, symbol Device:C
- added C15: 1uF, Capacitor_SMD:C_0805_2012Metric_Pad1.18x1.45mm_HandSolder, symbol Device:C_Small
- added C16: 100nF, Capacitor_SMD:C_0805_2012Metric_Pad1.18x1.45mm_HandSolder, symbol Device:C_Small
- added C3: 104, symbol Device:C
- added H1, H2, H3, H4: MountingHole, symbol Mechanical:MountingHole
- added J2: HC12, symbol Connector:Conn_01x04_Pin
- added J3: C1101, symbol Connector:Conn_01x06_Pin
- added J4: BNO055, symbol Connector:Conn_01x08_Pin
- added J6: ILI9341, symbol Connector:Conn_01x09_Pin
- added J7: DEBUG, symbol Connector:Conn_01x04_Pin
- added JP1, JP2: SolderJumper_3_Open, symbol Jumper:SolderJumper_3_Open
- added JP6: Jumper_3_Open, symbol Jumper:Jumper_3_Open
- added MOTOR1, MOTOR2, MOTOR3, MOTOR4: Conn_01x04_Pin, symbol Connector:Conn_01x04_Pin
- added R1, R2, R3, R4: 10K, symbol Device:R
- added R10: 120R, Resistor_SMD:R_0805_2012Metric_Pad1.20x1.40mm_HandSolder, symbol Device:R_Small
- added R7, R8, R9: 4K7, Resistor_SMD:R_0805_2012Metric_Pad1.20x1.40mm_HandSolder, symbol Device:R_Small
- added SW1: SW_Push, symbol Switch:SW_Push
- added U1: STM32G473RETx, Package_QFP:LQFP-64_10x10mm_P0.5mm, symbol MCU_ST_STM32G4:STM32G473RETx
- added U2: MAX3485, Package_SO:SOIC-8_3.9x4.9mm_P1.27mm, symbol Interface_UART:MAX3485
- added Y1: 8MHz, symbol Device:Crystal
Connections:
- new net: C2.2, U1.6 (PF1), Y1.1
- new net: JP6.1 (A), R4.2
- new net: C1.2, U1.5 (PF0), Y1.2
- new net +3.3V: C10.1, C15.1, C16.1, C3.1, J2.1 (Pin_1), J3.1 (Pin_1), J4.1 (Pin_1), J6.1 (Pin_1), J7.1 (Pin_1), MOTOR1.1 (Pin_1), MOTOR2.1 (Pin_1), MOTOR3.1 (Pin_1), MOTOR4.1 (Pin_1), R3.1, R4.1, R7.1, R8.1, U1.1 (VBAT), U1.16 (VDD), U1.29 (VDDA), U1.32 (VDD), U1.48 (VDD), U1.64 (VDD), U2.8 (VCC)
- new net +3V3: R1.1, R2.2
- new net ADD: J4.5 (Pin_5)
- new net A_485: JP1.1 (A), R10.1, U2.6 (A)
- new net BOOT: J4.7 (Pin_7), JP6.2 (C), U1.61 (PB8)
- new net B_485: JP2.1 (A), R10.2, U2.7 (B)
- new net CS_C1101: J3.3 (Pin_3)
- new net CS_TFT: J6.3 (Pin_3)
- new net DC: J6.5 (Pin_5)
- new net GND: C1.1, C10.2, C15.2, C16.2, C2.1, C3.2, J2.2 (Pin_2), J3.2 (Pin_2), J4.2 (Pin_2), J6.2 (Pin_2), J7.4 (Pin_4), JP6.3 (B), MOTOR1.4 (Pin_4), MOTOR2.4 (Pin_4), MOTOR3.4 (Pin_4), MOTOR4.4 (Pin_4), R9.2, SW1.1, U1.15 (VSS), U1.27 (VSSA), U1.31 (VSS), U1.47 (VSS), U1.63 (VSS), U2.5 (GND)
- new net INT: J4.6 (Pin_6)
- new net LED: J6.8 (Pin_8)
- new net MISO: J3.6 (Pin_6), J6.9 (Pin_9), U1.20 (PA6)
- new net MOSI: J3.5 (Pin_5), J6.6 (Pin_6), U1.21 (PA7)
- new net NRST: R3.2, SW1.2, U1.7 (PG10)
- new net OUT1: JP1.2 (C), MOTOR1.2 (Pin_2), MOTOR2.2 (Pin_2), MOTOR3.2 (Pin_2), MOTOR4.2 (Pin_2)
- new net OUT2: JP2.2 (C), MOTOR1.3 (Pin_3), MOTOR2.3 (Pin_3), MOTOR3.3 (Pin_3), MOTOR4.3 (Pin_3)
- new net RESET: J4.8 (Pin_8)
- new net RE_DE: R9.1, U2.2 (~{RE}), U2.3 (DE)
- new net RST: J6.4 (Pin_4)
- new net RX1: JP2.3 (B), U1.23 (PC5)
- new net RX2: R8.2, U1.17 (PA3), U2.1 (RO)
- new net RX3: J2.4 (Pin_4), U1.33 (PB11)
- new net SCK: J3.4 (Pin_4), J6.7 (Pin_7), U1.19 (PA5)
- new net SCL: J4.3 (Pin_3), R1.2, U1.60 (PB7)
- new net SDA: J4.4 (Pin_4), R2.1, U1.51 (PA15)
- new net SWCLK: J7.3 (Pin_3), U1.50 (PA14)
- new net SWDIO: J7.2 (Pin_2), U1.49 (PA13)
- new net TX1: JP1.3 (B), U1.22 (PC4)
- new net TX2: R7.2, U1.14 (PA2), U2.4 (DI)
- new net TX3: J2.3 (Pin_3), U1.30 (PB10)
Other:
- added sheet IO (Indicator.kicad_sch)
- added sheet Power (Power.kicad_sch)
