File: hardware/MAIN_CONTROLLER/Indicator.kicad_sch (KiCad schematic)
At the start: 37 parts, among them J8 Conn_01x11, Q1 AO3400A, U5 PCF8575DBR, U8 CD74HC4067M

Commit message: Schematic update
Parts:
- removed J8: Conn_01x11, symbol Connector_Generic:Conn_01x11
- added J8: Conn_01x16_Pin, symbol Connector:Conn_01x16_Pin
Connections:
- net +3.3V: no longer R13.2, R14.2, R15.2, R16.2, R17.2, R18.2, R19.2, R20.2, R21.2, R22.2, R23.2
- net GND: now also R13.2, R14.2, R15.2, R16.2, R17.2, R18.2, R19.2, R20.2, R21.2, R22.2, R23.2
- net at U8.16 (I15): now also J8.16 (Pin_16)
- net at U8.17 (I14): now also J8.15 (Pin_15)
- net at U8.18 (I13): now also J8.14 (Pin_14)
- net at U8.19 (I12): now also J8.13 (Pin_13)
- net at U8.2 (I7): now also J8.8 (Pin_8)
- net at U8.20 (I11): now also J8.12 (Pin_12)
- net at U8.21 (I10): now also J8.11 (Pin_11)
- net at U8.22 (I9): now also J8.10 (Pin_10)
- net at U8.23 (I8): now also J8.9 (Pin_9)
- net at U8.3 (I6): now also J8.7 (Pin_7)
- net at U8.4 (I5): now also J8.6 (Pin_6)
- net at U8.5 (I4): now also J8.5 (Pin_5)
- net at U8.6 (I3): now also J8.4 (Pin_4)
- net at U8.7 (I2): now also J8.3 (Pin_3)
- net at U8.8 (I1): now also J8.2 (Pin_2)
- net at U8.9 (I0): now also J8.1 (Pin_1)
- no-connect marks 11 -> 6
