File: hardware/MAIN_CONTROLLER/MAIN_CONTROLLER.kicad_sch (KiCad schematic)
At the start: 34 parts, among them J2 HC12, J3 C1101, J4 BNO055, J6 ILI9341, J7 DEBUG, SW1 SW_Push, U1 STM32G473RETx, U2 MAX3485, Y1 8MHz

Commit message: Schematic update
Parts:
- added J13: USB_C_Receptacle_USB2.0_16P, symbol Connector:USB_C_Receptacle_USB2.0_16P
Connections:
- net RE_DE: now also U1.18 (PA4)
- new net: J13.A1 (GND), J13.A12 (GND), J13.B1 (GND), J13.B12 (GND)
- new net: J13.A4 (VBUS), J13.A9 (VBUS), J13.B4 (VBUS), J13.B9 (VBUS)
Changed lines of the file:
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@@
 	(wire
 		(pts
+			(xy 115.57 57.15) (xy 119.38 57.15)
+		)
+		(stroke
+			(width 0)
+			(type default)
+		)
+	)
+	(wire
+		(pts
 			(xy 248.92 33.02) (xy 254 33.02)
 		)
@@
 		)
 	)
+	(label "RE_DE"
+		(at 119.38 57.15 0)
+		(effects
+			(font
+				(size 1.27 1.27)
+			)
+			(justify left bottom)
+		)
+	)
 	(label "OUT2"
 		(at 209.55 39.37 0)
@@
 					(unit 1)
 				)
+			)
+		)
+	)
+	(symbol
+		(lib_id "Connector:USB_C_Receptacle_USB2.0_16P")
+		(at 219.71 137.16 0)
+		(unit 1)
+		(body_style 1)
+		(exclude_from_sim no)
+		(in_bom yes)
+		(on_board yes)
+		(in_pos_files yes)
+		(dnp no)
+		(fields_autoplaced yes)
+		(property "Reference" "J13"
+			(at 219.71 114.3 0)
+			(show_name no)
+			(do_not_autoplace no)
+			(effects
+				(font
+					(size 1.27 1.27)
+				)
+			)
+		)
+		(property "Value" "USB_C_Receptacle_USB2.0_16P"
+			(at 219.71 116.84 0)
+			(show_name no)
+			(do_not_autoplace no)
+			(effects
+				(font
+					(size 1.27 1.27)
+				)
+			)
+		)
+		(property "Footprint" ""
+			(at 223.52 137.16 0)
+			(hide yes)
+			(show_name no)
+			(do_not_autoplace no)
+			(effects
+				(font
+					(size 1.27 1.27)
+				)
+			)
+		)
+		(property "Datasheet" "https://www.usb.org/sites/default/files/documents/usb_type-c.zip"
+			(at 223.52 137.16 0)
+			(hide yes)
+			(show_name no)
+			(do_not_autoplace no)
+			(effects
+				(font
+					(size 1.27 1.27)
+				)
+			)
+		)
+		(property "Description" "USB 2.0-only 16P Type-C Receptacle connector"
+			(at 219.71 137.16 0)
+			(hide yes)
+			(show_name no)
+			(do_not_autoplace no)
+			(effects
+				(font
+					(size 1.27 1.27)
+				)
+			)
+		)
+		(pin "B5"
+		)
+		(pin "B7"
+		)
+		(pin "A5"
+		)
+		(pin "A7"
+		)
+		(pin "B9"
+		)
+		(pin "A8"
+		)
+		(pin "B8"
+		)
+		(pin "SH"
+		)
+		(pin "A1"
+		)
+		(pin "A6"
+		)
+		(pin "A9"
+		)
+		(pin "A12"
+		)
+		(pin "A4"
+		)
+		(pin "B1"
+		)
+		(pin "B4"
+		)
+		(pin "B6"
+		)
+		(pin "B12"
+		)
+		(instances
+			(project "MAIN_CONTROLLER"
+				(path "/04ac99f1-194a-459d-a9b5-7c43d6ccc196"
+					(reference "J13")
+					(unit 1)
+				)
