File: hardware/LINE_BOARD/mach_do_line/mach_do_line.kicad_sch (KiCad schematic)
At the start: 36 parts, among them J10 Conn_01x01_Pin, J11 Conn_01x01_Pin, J12 Conn_01x01_Pin, J13 Conn_01x01_Pin, J14 Conn_01x01_Pin, J15 Conn_01x01_Pin, J16 Conn_01x01_Pin, J17 Conn_01x01_Pin, J18 Conn_01x01_Pin, J2 Conn_01x01_Pin, J3 Conn_01x01_Pin, U2 RPR-220, U3 RPR-220, U4 RPR-220, U5 RPR-220, U6 RPR-220

Commit message: add pcb line
Parts:
- removed H3, H4: MountingHole, MountingHole:MountingHole_2.2mm_M2_ISO14580_Pad_TopBottom, symbol Mechanical:MountingHole
Changed lines of the file:
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@@
-	)
-	(symbol
-		(lib_id "Mechanical:MountingHole")
-		(at 173.99 165.1 0)
-		(unit 1)
-		(body_style 1)
-		(exclude_from_sim no)
-		(in_bom no)
-		(on_board yes)
-		(in_pos_files yes)
-		(dnp no)
-		(fields_autoplaced yes)
-		(property "Reference" "H4"
-			(at 176.53 163.8299 0)
-			(show_name no)
-			(do_not_autoplace no)
-			(effects
-				(font
-					(size 1.27 1.27)
-				)
-				(justify left)
-			)
-		)
-		(property "Value" "MountingHole"
-			(at 176.53 166.3699 0)
-			(show_name no)
-			(do_not_autoplace no)
-			(effects
-				(font
-					(size 1.27 1.27)
-				)
-				(justify left)
-			)
-		)
-		(property "Footprint" "MountingHole:MountingHole_2.2mm_M2_ISO14580_Pad_TopBottom"
-			(at 173.99 165.1 0)
-			(hide yes)
-			(show_name no)
-			(do_not_autoplace no)
-			(effects
-				(font
-					(size 1.27 1.27)
-				)
-			)
-		)
-		(property "Datasheet" ""
-			(at 173.99 165.1 0)
-			(hide yes)
-			(show_name no)
-			(do_not_autoplace no)
-			(effects
-				(font
-					(size 1.27 1.27)
-				)
-			)
-		)
-		(property "Description" "Mounting Hole without connection"
-			(at 173.99 165.1 0)
-			(hide yes)
-			(show_name no)
-			(do_not_autoplace no)
-			(effects
-				(font
-					(size 1.27 1.27)
-				)
-			)
-		)
-		(instances
-			(project "mach_do_line"
-				(path "/8d8fc8c2-eeac-4400-9949-5e185cac9288"
-					(reference "H4")
-					(unit 1)
-				)
-			)
-		)
 	)
 	(symbol
@@
 					(unit 1)
 				)
-			)
-		)
-	)
-	(symbol
-		(lib_id "Mechanical:MountingHole")
-		(at 152.4 163.83 0)
-		(unit 1)
-		(body_style 1)
-		(exclude_from_sim no)
-		(in_bom no)
-		(on_board yes)
-		(in_pos_files yes)
-		(dnp no)
-		(fields_autoplaced yes)
-		(property "Reference" "H3"
-			(at 154.94 162.5599 0)
-			(show_name no)
-			(do_not_autoplace no)
-			(effects
-				(font
-					(size 1.27 1.27)
-				)
-				(justify left)
-			)
-		)
-		(property "Value" "MountingHole"
-			(at 154.94 165.0999 0)
-			(show_name no)
-			(do_not_autoplace no)
-			(effects
-				(font
-					(size 1.27 1.27)
-				)
-				(justify left)
-			)
-		)
-		(property "Footprint" "MountingHole:MountingHole_2.2mm_M2_ISO14580_Pad_TopBottom"
-			(at 152.4 163.83 0)
-			(hide yes)
-			(show_name no)
-			(do_not_autoplace no)
-			(effects
-				(font
-					(size 1.27 1.27)
-				)
-			)
-		)
-		(property "Datasheet" ""
-			(at 152.4 163.83 0)
-			(hide yes)
-			(show_name no)
-			(do_not_autoplace no)
-			(effects
-				(font
-					(size 1.27 1.27)
-				)
-			)
-		)
-		(property "Description" "Mounting Hole without connection"
-			(at 152.4 163.83 0)
-			(hide yes)
-			(show_name no)
-			(do_not_autoplace no)
-			(effects
-				(font
-					(size 1.27 1.27)
-				)
-			)
-		)
-		(instances
-			(project "mach_do_line"
-				(path "/8d8fc8c2-eeac-4400-9949-5e185cac9288"
-					(reference "H3")
-					(unit 1)
-				)

Commit message: add pcb line 15mm, 10mm
Parts:
- removed C1: 220u, Capacitor_SMD:CP_Elec_4x3, symbol Device:C_Polarized_Small
- added C1, C2, C3, C4, C5, C6: 100uF, Capacitor_SMD:C_1206_3216Metric, symbol Device:C_Small
- added D1, D2, D3, D4, D5, D6: LED_Small, LED_SMD:LED_1206_3216Metric_Pad1.42x1.75mm_HandSolder, symbol Device:LED_Small
- added R1, R18, R19, R2, R20, R21: 220, Resistor_SMD:R_0805_2012Metric, symbol Device:R_Small
- U2, U3, U4, U5, U6: footprint RPR220:RPR220 -> RPR-220:RPR220
Connections:
- net +5V: now also C1.1, C2.1, C3.1, C4.1, C5.1, C6.1, D1.2 (A), D2.2 (A), D3.2 (A), D4.2 (A), D5.2 (A), D6.2 (A)
- net GND: now also C1.2, C2.2, C3.2, C4.2, C5.2, C6.2, R1.2, R18.2, R19.2, R2.2, R20.2, R21.2
- new net: D3.1 (K), R18.1
- new net: D4.1 (K), R19.1
- new net: D2.1 (K), R2.1
- new net: D5.1 (K), R20.1
- new net: D1.1 (K), R1.1
- new net: D6.1 (K), R21.1
